Commit message: add panda arm urdf with peg addition. WIP to get FT sensor and transform tip frame

File: robots/panda.gazebo.xacro (robot description, xacro)
@@ -1,5 +1,5 @@
 <?xml version="1.0"?>
 <robot xmlns:xacro="http://www.ros.org/wiki/xacro">
-    <xacro:macro name="panda_gazebo" params="robot_name load_gripper">
+    <xacro:macro name="panda_gazebo" params="robot_name load_peg load_gripper">
       <gazebo reference="${robot_name}_joint7">
         <implicitSpringDamper>1</implicitSpringDamper>
@@ -30,4 +30,11 @@
         <provideFeedback>true</provideFeedback>
       </gazebo>
+      <xacro:if value="${load_peg}">
+          <gazebo reference="${robot_name}_peg">
+            <material>Gazebo/Grey</material>
+            <mu1>100.0</mu1>
+            <mu2>100.0</mu2>
+          </gazebo>
+      </xacro:if>
       <xacro:if value="${load_gripper}">
           <gazebo reference="${robot_name}_finger_joint1">
@@ -41,4 +48,45 @@
       </xacro:if>
     <!-- Adding FT sensor at wrist. This is not present in real robot and is used only for computing end-point effort directly, unlike in the real robot where it is estimated from the joint efforts. -->
+    <!-- <xacro:if value="${load_peg}">
+      <gazebo reference="${robot_name}_peg_joint">
+        <disableFixedJointLumping>true</disableFixedJointLumping>
+        <sensor name="${robot_name}_peg_joint_force_torque" type="force_torque">
+          <always_on>true</always_on>
+          <visualize>false</visualize>
+          <force_torque>
+            <frame>sensor</frame>
+            <measure_direction>child_to_parent</measure_direction>
+          </force_torque>
+        </sensor>
+      </gazebo>
+      <gazebo>
+        <plugin name="ft_sensor" filename="libgazebo_ros_ft_sensor.so">
+          <updateRate>30.0</updateRate>
+          <topicName>/gazebo/robot/wrist/ft</topicName>
+          <jointName>panda_peg_joint</jointName>
+        </plugin>
+      </gazebo>
+    </xacro:if>
+    <xacro:if value="${load_gripper}">
+      <gazebo reference="${robot_name}_hand_joint">
+        <disableFixedJointLumping>true</disableFixedJointLumping>
+        <sensor name="${robot_name}_hand_joint_force_torque" type="force_torque">
+          <always_on>true</always_on>
+          <visualize>false</visualize>
+          <force_torque>
+            <frame>sensor</frame>
+            <measure_direction>child_to_parent</measure_direction>
+          </force_torque>
+        </sensor>
+      </gazebo>
+      <gazebo>
+        <plugin name="ft_sensor" filename="libgazebo_ros_ft_sensor.so">
+          <updateRate>30.0</updateRate>
+          <topicName>/gazebo/robot/wrist/ft</topicName>
+          <jointName>panda_hand_joint</jointName>
+        </plugin>
+      </gazebo>
+    </xacro:if> -->
+    <!-- previous ft sensor definition -->
     <gazebo reference="${robot_name}_joint7">
       <disableFixedJointLumping>true</disableFixedJointLumping>

File: robots/panda_arm_hand_peg.urdf.xacro (robot description, xacro)
@@ -2,5 +2,6 @@
 <robot xmlns:xacro="http://www.ros.org/wiki/xacro" name="panda">
   <xacro:arg name="robot_name" default="panda"/>
-  <xacro:arg name="load_gripper" default="true"/>
+  <xacro:arg name="load_gripper" default="false"/>
+  <xacro:arg name="load_peg" default="true"/>
   <xacro:arg name="load_gazebo" default="false"/>
   <xacro:arg name="use_gazebo_control" default="false"/>
@@ -11,9 +12,13 @@
     <xacro:hand ns="panda" rpy="0 0 ${-pi/4}" connected_to="panda_link8"/>
   </xacro:if>
+  <xacro:if value="$(arg load_peg)">
+    <xacro:include filename="$(find franka_panda_description)/robots/peg.xacro"/>
+    <xacro:peg ns="panda" rpy="0 0 ${-pi/4}" connected_to="panda_link8"/>
+  </xacro:if>
   <xacro:if value="$(arg load_gazebo)">
     <xacro:include filename="$(find franka_panda_description)/robots/panda.gazebo.xacro"/>
     <xacro:include filename="$(find franka_panda_description)/robots/panda.transmission.xacro"/>
     <xacro:panda_arm in_gazebo="true"  connected_to="$(arg connected_to)"/>
-    <xacro:panda_gazebo robot_name="$(arg robot_name)" load_gripper="$(arg load_gripper)"/>
+    <xacro:panda_gazebo robot_name="$(arg robot_name)" load_peg="$(arg load_peg)" load_gripper="$(arg load_gripper)"/>
     <xacro:panda_transmission robot_name="$(arg robot_name)" load_gripper="$(arg load_gripper)" use_gazebo_control="$(arg use_gazebo_control)"/>
   </xacro:if>
